File: hardware/kicad/tank-driver-recovery.kicad_sch (KiCad schematic)
At the start: 19 parts, among them J101 Primary L send, J102 Primary L return, J103 Primary R send, J104 Primary R return, J105 Secondary L send, J106 Secondary L return, J107 Secondary R send, J108 Secondary R return, P101 JTR-PRI, P102 JTR-SEC, P103 JTR-PWR, Q101 BD139-16, Q102 BD140-16, Q103 BD139-16, Q104 BD140-16, U101 OPA1656IDR, U102 OPA1656IDR, U103 OPA1656IDR, U104 OPA1656IDR

Commit message: Rebuild tank-driver-recovery: ERC-clean schematic + working ngspice testbench + netlist-synced placed PCB (DRC errors 0, routing pending)
Parts:
- added C101, C121: 47n, Capacitor_SMD:C_1210_3225Metric, symbol Device:C
- added C171, C172, C173, C174: 68p, Capacitor_SMD:C_0805_2012Metric, symbol Device:C
- added C175, C176, C177, C178: 22n, Capacitor_SMD:C_1206_3216Metric, symbol Device:C
- added C191: 1n, Capacitor_SMD:C_0805_2012Metric, symbol Device:C
- added C291, C292, C293, C294, C295, C296, C297, C298: 100n, Capacitor_SMD:C_0805_2012Metric, symbol Device:C
- added C299, C300: 22u, Capacitor_SMD:C_1210_3225Metric, symbol Device:C
- added D101, D102, D121, D122: 1N4148W, Diode_SMD:D_SOD-123, symbol Device:D
- added R101, R102, R121, R122: 68, Resistor_SMD:R_0805_2012Metric, symbol Device:R
- added R103, R104, R123, R124: 0.33, Resistor_SMD:R_2512_6332Metric, symbol Device:R
- added R105, R125: 10, Resistor_SMD:R_1206_3216Metric, symbol Device:R
- added R106, R126, R175, R176, R177, R178: 1k, Resistor_SMD:R_0805_2012Metric, symbol Device:R
- added R107, R108, R127, R128, R153, R154, R157, R158: 10k, Resistor_SMD:R_0805_2012Metric, symbol Device:R
- added R151, R152: 12k, Resistor_SMD:R_0805_2012Metric, symbol Device:R
- added R155, R156: 220, Resistor_SMD:R_0805_2012Metric, symbol Device:R
- added R171, R172, R173, R174: 2.2Meg, Resistor_SMD:R_0805_2012Metric, symbol Device:R
- added R179, R180, R181, R182: 33k, Resistor_SMD:R_0805_2012Metric, symbol Device:R
- added R183, R184, R185, R186: 0, Resistor_SMD:R_0805_2012Metric, symbol Device:R
- added R205: 100, Resistor_SMD:R_1206_3216Metric, symbol Device:R
- added R206: 0, Resistor_SMD:R_1206_3216Metric, symbol Device:R
- added unit 3 of U101
- added unit 2 of U101
- added unit 2 of U102
- added unit 3 of U102
- added unit 2 of U103
- added unit 3 of U103
- added unit 2 of U104
- added unit 3 of U104
- J101: value Primary L send -> PRI L SEND; footprint (none) -> Connector_JST:JST_XH_B2B-XH-A_1x02_P2.50mm_Vertical
- J102: value Primary L return -> PRI L RET; footprint (none) -> Connector_JST:JST_XH_B2B-XH-A_1x02_P2.50mm_Vertical
- J103: value Primary R send -> PRI R SEND; footprint (none) -> Connector_JST:JST_XH_B2B-XH-A_1x02_P2.50mm_Vertical
- J104: value Primary R return -> PRI R RET; footprint (none) -> Connector_JST:JST_XH_B2B-XH-A_1x02_P2.50mm_Vertical
- J105: value Secondary L send -> SEC L SEND; footprint (none) -> Connector_JST:JST_XH_B2B-XH-A_1x02_P2.50mm_Vertical
- J106: value Secondary L return -> SEC L RET; footprint (none) -> Connector_JST:JST_XH_B2B-XH-A_1x02_P2.50mm_Vertical
- J107: value Secondary R send -> SEC R SEND; footprint (none) -> Connector_JST:JST_XH_B2B-XH-A_1x02_P2.50mm_Vertical
- J108: value Secondary R return -> SEC R RET; footprint (none) -> Connector_JST:JST_XH_B2B-XH-A_1x02_P2.50mm_Vertical
- P101: value JTR-PRI -> JTR-PRI B6B-XH-A
- P102: value JTR-SEC -> JTR-SEC B6B-XH-A
- P103: value JTR-PWR -> JTR-PWR B3P-VH-B
Connections:
- net PRI_RET_L: now also P101.2 (Pin_2), U103.1, C171.1, R179.1
- net PRI_RET_R: now also P101.5 (Pin_5), C172.1, R180.1, U103.7
- net PRI_SEND_L: now also P101.1 (Pin_1), R106.1, R107.1
- net PRI_SEND_R: now also P101.4 (Pin_4), R126.1, R127.1
- net SEC_RET_L: now also P102.2 (Pin_2), U104.1, C173.1, R181.1
- net SEC_RET_R: now also P102.5 (Pin_5), C174.1, R182.1, U104.7
- net SEC_SEND_L: now also P102.1 (Pin_1), R157.1
- net SEC_SEND_R: now also P102.4 (Pin_4), R158.1
- new net +15VA: C291.1, C292.1, C293.1, C294.1, C299.1, P103.1 (Pin_1), Q101.2 (C), Q103.2 (C), U101.8 (V+), U102.8 (V+), U103.8 (V+), U104.8 (V+)
- new net -15VA: C295.1, C296.1, C297.1, C298.1, C300.1, P103.3 (Pin_3), Q102.2 (C), Q104.2 (C), U101.4 (V-), U102.4 (V-), U103.4 (V-), U104.4 (V-)
- new net AGND: C101.2, C121.2, C191.2, C291.2, C292.2, C293.2, C294.2, C295.2, C296.2, C297.2, C298.2, C299.2, C300.2, P101.3 (Pin_3), P101.6 (Pin_6), P102.3 (Pin_3), P102.6 (Pin_6), P103.2 (Pin_2), R153.2, R154.2, R171.2, R172.2, R173.2, R174.2, R175.2, R176.2, R177.2, R178.2, R205.2
- new net N_PRI_L_M: R106.2, R108.2, U101.2 (-)
- new net N_PRI_L_P: R107.2, U101.3 (+)
- new net N_PRI_RET_L_M: C171.2, R175.1, R179.2, U103.2 (-)
- new net N_PRI_RET_R_M: C172.2, R176.1, R180.2, U103.6 (-)
- new net N_PRI_R_M: R126.2, R128.2, U101.6 (-)
- new net N_PRI_R_P: R127.2, U101.5 (+)
- new net N_Q101_B: D101.2 (A), Q101.3 (B), R101.2
- new net N_Q101_E: Q101.1 (E), R103.1
- new net N_Q102_B: D102.1 (K), Q102.3 (B), R102.2
- new net N_Q102_E: Q102.1 (E), R104.1
- new net N_Q103_B: D121.2 (A), Q103.3 (B), R121.2
- new net N_Q103_E: Q103.1 (E), R123.1
- new net N_Q104_B: D122.1 (K), Q104.3 (B), R122.2
- new net N_Q104_E: Q104.1 (E), R124.1
- new net N_REC_PL_IN: C175.2, R183.2, U103.3 (+)
- new net N_REC_PR_IN: C176.2, R184.2, U103.5 (+)
- new net N_REC_SL_IN: C177.2, R185.2, U104.3 (+)
- new net N_REC_SR_IN: C178.2, R186.2, U104.5 (+)
- new net N_SEC_L_M: R151.2, R153.1, U102.2 (-)
- new net N_SEC_L_P: R157.2, U102.3 (+)
- new net N_SEC_RET_L_M: C173.2, R177.1, R181.2, U104.2 (-)
- new net N_SEC_RET_R_M: C174.2, R178.1, R182.2, U104.6 (-)
- new net N_SEC_R_M: R152.2, R154.1, U102.6 (-)
- new net N_SEC_R_P: R158.2, U102.5 (+)
- new net N_ZOB_L: C101.1, R105.2
- new net N_ZOB_R: C121.1, R125.2
- new net PRI_DRV_L: D101.1 (K), D102.2 (A), R101.1, R102.1, U101.1
- new net PRI_DRV_R: D121.1 (K), D122.2 (A), R121.1, R122.1, U101.7
- new net PRI_OUT_L: J101.1 (In), R103.2, R104.2, R105.1, R108.1
- new net PRI_OUT_R: J103.1 (In), R123.2, R124.2, R125.1, R128.1
- new net PRI_REC_L_IN: C175.1, J102.1 (In), R171.1, R183.1
- new net PRI_REC_R_IN: C176.1, J104.1 (In), R172.1, R184.1
- new net SEC_DRV_L: R151.1, R155.1, U102.1
- new net SEC_DRV_R: R152.1, R156.1, U102.7
- new net SEC_OUT_L: J105.1 (In), R155.2
- new net SEC_OUT_R: J107.1 (In), R156.2
- new net SEC_REC_L_IN: C177.1, J106.1 (In), R173.1, R185.1
- new net SEC_REC_R_IN: C178.1, J108.1 (In), R174.1, R186.1
- new net TANK_SHIELD_RET: C191.1, J102.2 (Ext), J104.2 (Ext), J106.2 (Ext), J108.2 (Ext), R205.1, R206.2
- new net TANK_SHIELD_SEND: J101.2 (Ext), J103.2 (Ext), J105.2 (Ext), J107.2 (Ext), R206.1
Other:
- note added: "BOARD HARNESS"
- note added: "POWER ENTRY + DECOUPLING"
- note added: "PRIMARY SEND LEFT (4AB1C1B, 8R)"
- note added: "PRIMARY SEND RIGHT (4AB1C1B, 8R)"
- note added: "RECOVERY PRIMARY L"
- note added: "RECOVERY PRIMARY R"
- note added: "RECOVERY SECONDARY L"
- note added: "RECOVERY SECONDARY R"
- note added: "SECONDARY SENDS (9EB2C1B L / 9EB3C1B R, 800R)"
- note added: "TANK SHIELD STRATEGY"
- note removed: "Routing and power headers"
- note removed: "Send and recovery devices"
- note removed: "Tank board first-pass symbol capture - All required board refs are now present as real KiCad symbols - Tank send/return landings are captured as provisional coaxial connectors pending final RCA or shielded-wire hardware freeze - Primary driver bias parts, recovery gain networks, and exact shield strategy still need the next capture pass"
- note removed: "Tank cable landings"
