File: hardware/kicad/tank-driver-recovery.kicad_sch (KiCad schematic)
At the start: 19 parts, among them J101 Primary L send, J102 Primary L return, J103 Primary R send, J104 Primary R return, J105 Secondary L send, J106 Secondary L return, J107 Secondary R send, J108 Secondary R return, P101 JTR-PRI, P102 JTR-SEC, P103 JTR-PWR, Q101 BD139-16, Q102 BD140-16, Q103 BD139-16, Q104 BD140-16, U101 OPA1656IDR, U102 OPA1656IDR, U103 OPA1656IDR, U104 OPA1656IDR

Commit message: Rev A: 3-pass schematic review + fixes, PCB sync + placement, parts freeze (2026-07-31)
Pass1+2 fixed cross-channel shorts (io rails/C1-C4/alias columns), ext-tank ghost wiring, U201 unit un-stack, U101-104 power units, PS500 pinout from datasheet, DRV renames. Decisions: TQ2-5V relays +D301, R241-3 deleted, PGND_IN+R502 link, K401-403 clip decoder, RCJ-041 tank jacks. GAS_Parts lib (TQ2/URA_YMD/RCJ-041), ~203 footprints, 6 boards synced+placed DRC-clean. Pass3 visual: paper sizes, stale notes. 3D GLBs + viewer. See hardware/kicad/schematic_review.md
Parts:
- added C101, C102, C104, C201, C202, C204, C301, C302, C304, C401, C402, C404: 10uF, Capacitor_SMD:CP_Elec_5x5.8, symbol Device:C
- added C103, C203, C303, C403: 220pF, Capacitor_SMD:C_0603_1608Metric, symbol Device:C
- added D101, D102, D201, D202, D301, D302, D401, D402: 1N4148, Diode_SMD:D_SOD-123, symbol Device:D
- added Q105, Q107: BD139-16, Package_TO_SOT_THT:TO-126-3_Vertical, symbol Transistor_BJT:BD139
- added Q106, Q108: BD140-16, Package_TO_SOT_THT:TO-126-3_Vertical, symbol Transistor_BJT:BD140
- added R101, R201, R301, R401: 10k, Resistor_SMD:R_0603_1608Metric, symbol Device:R
- added R102, R105, R106, R202, R205, R206, R302, R305, R306, R402, R405, R406: 100R, Resistor_SMD:R_0603_1608Metric, symbol Device:R
- added R103, R104, R112, R203, R204, R212, R303, R304, R312, R403, R404, R412: 2.2k, Resistor_SMD:R_0603_1608Metric, symbol Device:R
- added R107, R108, R207, R208, R307, R308, R407, R408: 10R, Resistor_SMD:R_1206_3216Metric, symbol Device:R
- added R109, R113, R209, R213, R309, R313, R409, R413: 1k, Resistor_SMD:R_0603_1608Metric, symbol Device:R
- added R110, R210, R310, R410: 47R, Resistor_SMD:R_0603_1608Metric, symbol Device:R
- added R111, R115, R211, R215, R311, R315, R411, R415: 100k, Resistor_SMD:R_0603_1608Metric, symbol Device:R
- added R114, R214, R314, R414: 47k, Resistor_SMD:R_0603_1608Metric, symbol Device:R
- added unit 3 of U101
- added unit 2 of U101
- added unit 2 of U102
- added unit 3 of U102
- added unit 2 of U103
- added unit 3 of U103
- added unit 3 of U104
- added unit 2 of U104
- J101, J102, J103, J104, J105, J106, J107, J108: footprint (none) -> GAS_Parts:Jack_RCA_SameSky_RCJ-041_Horizontal; MPN (none) -> RCJ-041
Connections:
- net PRI_RET_L: now also P101.4 (Pin_4), C104.2, R115.1
- net PRI_RET_R: now also P101.1 (Pin_1), C204.2, R215.1
- net PRI_SEND_L: now also P101.5 (Pin_5), C101.1
- net PRI_SEND_R: now also P101.2 (Pin_2), C201.1
- net SEC_RET_L: now also P102.4 (Pin_4), C304.2, R315.1
- net SEC_RET_R: now also P102.1 (Pin_1), C404.2, R415.1
- net SEC_SEND_L: now also P102.5 (Pin_5), C301.1
- net SEC_SEND_R: now also P102.2 (Pin_2), C401.1
- new net +15VA: P103.1 (Pin_1), Q101.2 (C), Q103.2 (C), Q105.2 (C), Q107.2 (C), R103.1, R203.1, R303.1, R403.1, U101.8 (V+), U102.8 (V+), U103.8 (V+), U104.8 (V+)
- new net -15VA: P103.3 (Pin_3), Q102.2 (C), Q104.2 (C), Q106.2 (C), Q108.2 (C), R104.2, R204.2, R304.2, R404.2, U101.4 (V-), U102.4 (V-), U103.4 (V-), U104.4 (V-)
- new net AGND: J101.2 (Ext), J102.2 (Ext), J103.2 (Ext), J104.2 (Ext), J105.2 (Ext), J106.2 (Ext), J107.2 (Ext), J108.2 (Ext), P101.3 (Pin_3), P101.6 (Pin_6), P102.3 (Pin_3), P102.6 (Pin_6), P103.2 (Pin_2), R101.2, R111.2, R112.2, R113.2, R115.2, R201.2, R211.2, R212.2, R213.2, R215.2, R301.2, R311.2, R312.2, R313.2, R315.2, R401.2, R411.2, R412.2, R413.2, R415.2
- new net PL_BIAS_A: D101.2 (A), R103.2, R105.1
- new net PL_BIAS_B: D102.1 (K), R104.1, R106.1
- new net PL_BIAS_MID: D101.1 (K), D102.2 (A), R102.2
- new net PL_DRV_FB: R109.2, U101.2 (-)
- new net PL_DRV_IN: C101.2, R101.1, U101.3 (+)
- new net PL_DRV_OUT: R102.1, U101.1
- new net PL_J102_IN: C102.1, J102.1 (In), R112.1
- new net PL_Q101_B: Q101.3 (B), R105.2
- new net PL_Q101_E: Q101.1 (E), R107.1
- new net PL_Q102_B: Q102.3 (B), R106.2
- new net PL_Q102_E: Q102.1 (E), R108.1
- new net PL_REC_FB: C103.2, R113.1, R114.2, U101.6 (-)
- new net PL_REC_IN: C102.2, R111.1, U101.5 (+)
- new net PL_REC_OUT: C103.1, C104.1, R114.1, U101.7
- new net PL_TANK: R107.2, R108.2, R109.1, R110.1
- new net PL_TANK_OUT: J101.1 (In), R110.2
- new net PR_BIAS_A: D201.2 (A), R203.2, R205.1
- new net PR_BIAS_B: D202.1 (K), R204.1, R206.1
- new net PR_BIAS_MID: D201.1 (K), D202.2 (A), R202.2
- new net PR_DRV_FB: R209.2, U102.2 (-)
- new net PR_DRV_IN: C201.2, R201.1, U102.3 (+)
- new net PR_DRV_OUT: R202.1, U102.1
- new net PR_J104_IN: C202.1, J104.1 (In), R212.1
- new net PR_Q103_B: Q103.3 (B), R205.2
- new net PR_Q103_E: Q103.1 (E), R207.1
- new net PR_Q104_B: Q104.3 (B), R206.2
- new net PR_Q104_E: Q104.1 (E), R208.1
- new net PR_REC_FB: C203.2, R213.1, R214.2, U102.6 (-)
- new net PR_REC_IN: C202.2, R211.1, U102.5 (+)
- new net PR_REC_OUT: C203.1, C204.1, R214.1, U102.7
- new net PR_TANK: R207.2, R208.2, R209.1, R210.1
- new net PR_TANK_OUT: J103.1 (In), R210.2
- new net SL_BIAS_A: D301.2 (A), R303.2, R305.1
- new net SL_BIAS_B: D302.1 (K), R304.1, R306.1
- new net SL_BIAS_MID: D301.1 (K), D302.2 (A), R302.2
- new net SL_DRV_FB: R309.2, U103.2 (-)
- new net SL_DRV_IN: C301.2, R301.1, U103.3 (+)
- new net SL_DRV_OUT: R302.1, U103.1
- new net SL_J106_IN: C302.1, J106.1 (In), R312.1
- new net SL_Q105_B: Q105.3 (B), R305.2
- new net SL_Q105_E: Q105.1 (E), R307.1
- new net SL_Q106_B: Q106.3 (B), R306.2
- new net SL_Q106_E: Q106.1 (E), R308.1
- new net SL_REC_FB: C303.2, R313.1, R314.2, U103.6 (-)
- new net SL_REC_IN: C302.2, R311.1, U103.5 (+)
- new net SL_REC_OUT: C303.1, C304.1, R314.1, U103.7
- new net SL_TANK: R307.2, R308.2, R309.1, R310.1
- new net SL_TANK_OUT: J105.1 (In), R310.2
- new net SR_BIAS_A: D401.2 (A), R403.2, R405.1
- new net SR_BIAS_B: D402.1 (K), R404.1, R406.1
- new net SR_BIAS_MID: D401.1 (K), D402.2 (A), R402.2
- new net SR_DRV_FB: R409.2, U104.2 (-)
- new net SR_DRV_IN: C401.2, R401.1, U104.3 (+)
- new net SR_DRV_OUT: R402.1, U104.1
- new net SR_J108_IN: C402.1, J108.1 (In), R412.1
- new net SR_Q107_B: Q107.3 (B), R405.2
- new net SR_Q107_E: Q107.1 (E), R407.1
- new net SR_Q108_B: Q108.3 (B), R406.2
- new net SR_Q108_E: Q108.1 (E), R408.1
- new net SR_REC_FB: C403.2, R413.1, R414.2, U104.6 (-)
- new net SR_REC_IN: C402.2, R411.1, U104.5 (+)
- new net SR_REC_OUT: C403.1, C404.1, R414.1, U104.7
- new net SR_TANK: R407.2, R408.2, R409.1, R410.1
- new net SR_TANK_OUT: J107.1 (In), R410.2
Other:
- note added: "Tank board first-pass symbol capture - All required board refs are now present as real KiCad symbols - Tank send/return landings FROZEN 2026-07-31: Same Sky RCJ-041 board-mount RCA jacks (shield=sleeve to AGND at each jack) - COMPLETE 2026-07-31: bias parts, recovery networks, and op-amp power units all placed & verified (see schematic_review.md)"
- note removed: "Tank board first-pass symbol capture - All required board refs are now present as real KiCad symbols - Tank send/return landings are captured as provisional coaxial connectors pending final RCA or shielded-wire hardware freeze - Primary driver bias parts, recovery gain networks, and exact shield strategy still need the next capture pass"
