File: hardware/kicad/crossfade-feedback-wet.kicad_sch (KiCad schematic)
At the start: 8 parts, among them P301 JTR-XFADE, P302 JXF-FILT, P303 JFILT-WET, P304 JIO-WETRET, P305 JFB-INJ, P306 JXFD-PWR, P307 JXFD-CTRL, U301 OPA1679IDR

Commit message: Board 3 crossfade-feedback-wet: ERC 0, sim verified (crossfade/wet/feedback math exact), routed DRC 0/0, fab outputs; added K301 G5V-2 phase-select relay missing from old BOM
Parts:
- added C321, C322: 47p, Capacitor_SMD:C_0805_2012Metric, symbol Device:C
- added C391, C392: 100n, Capacitor_SMD:C_0805_2012Metric, symbol Device:C
- added C393, C394: 22u, Capacitor_SMD:C_1210_3225Metric, symbol Device:C
- added D301: 1N4148W, Diode_SMD:D_SOD-123, symbol Device:D
- added K301: G5V-2 12VDC, Relay_THT:Relay_DPDT_Omron_G5V-2, symbol Relay:G5V-2
- added R301, R302, R309, R310, R321, R322, R323, R324: 20k, Resistor_SMD:R_0805_2012Metric, symbol Device:R
- added R311, R312, R331, R332, R341, R342: 100, Resistor_SMD:R_0805_2012Metric, symbol Device:R
- added R325, R326: 10k, Resistor_SMD:R_0805_2012Metric, symbol Device:R
- added R351: 240, Resistor_SMD:R_1206_3216Metric, symbol Device:R
- added unit 5 of U301
- added unit 2 of U301
- added unit 3 of U301
- added unit 4 of U301
- P301: value JTR-XFADE -> P301
- P302: value JXF-FILT -> P302
- P303: value JFILT-WET -> P303
- P304: value JIO-WETRET -> P304
- P305: value JFB-INJ -> P305
- P306: value JXFD-PWR -> JXFD-PWR B3P-VH-B
- P307: value JXFD-CTRL -> P307
Connections:
- net CTL_FB_INV: now also P307.9 (Pin_9), D301.2 (A), K301.16
- net FB_L_WIPER: now also P307.7 (Pin_7), R323.1
- net FB_RET_L: now also P305.1 (Pin_1), R331.2
- net FB_RET_R: now also P305.3 (Pin_3), R332.2
- net FB_R_WIPER: now also P307.8 (Pin_8), R324.1
- net FILTCLIP_OUT_L: now also P303.1 (Pin_1), K301.6, R321.1, R341.1
- net FILTCLIP_OUT_R: now also P303.3 (Pin_3), K301.11, R322.1, R342.1
- net TANK_MIX_L: now also P301.1 (Pin_1), P307.1 (Pin_1), P307.6 (Pin_6)
- net TANK_MIX_R: now also P301.3 (Pin_3), P307.3 (Pin_3), P307.4 (Pin_4)
- net WET_SUM_L: now also P304.1 (Pin_1), R341.2
- net WET_SUM_R: now also P304.3 (Pin_3), R342.2
- net XFADE_OUT_L: now also P302.1 (Pin_1), R311.2
- net XFADE_OUT_R: now also P302.3 (Pin_3), R312.2
- net XFD_L_WIPER: now also P307.2 (Pin_2), R301.1
- net XFD_R_WIPER: now also P307.5 (Pin_5), R302.1
- new net +15VA: C391.1, C393.1, P306.1 (Pin_1), R351.1, U301.4 (V+)
- new net -15VA: C392.1, C394.1, P306.3 (Pin_3), U301.11 (V-)
- new net AGND: C391.2, C392.2, C393.2, C394.2, P301.2 (Pin_2), P302.2 (Pin_2), P303.2 (Pin_2), P304.2 (Pin_2), P305.2 (Pin_2), P306.2 (Pin_2), P307.10 (Pin_10), U301.10 (+), U301.12 (+), U301.3 (+), U301.5 (+)
- new net FB_INV_L: C321.1, K301.8, R325.1, U301.8
- new net FB_INV_R: C322.1, K301.9, R326.1, U301.14
- new net FB_SEL_L: K301.4, R331.1
- new net FB_SEL_R: K301.13, R332.1
- new net N_FB_L_M: C321.2, R321.2, R323.2, R325.2, U301.9 (-)
- new net N_FB_R_M: C322.2, R322.2, R324.2, R326.2, U301.13 (-)
- new net N_K301_C: D301.1 (K), K301.1, R351.2
- new net N_XF_L_M: R301.2, R309.2, U301.2 (-)
- new net N_XF_R_M: R302.2, R310.2, U301.6 (-)
- new net XFADE_SUM_L: R309.1, R311.1, U301.1
- new net XFADE_SUM_R: R310.1, R312.1, U301.7
Other:
- note added: "CROSSFADE SUMMERS (U301A/B, inverting, unity)"
- note added: "FEEDBACK DRIVERS (U301C/D, inverting)"
- note added: "FEEDBACK PHASE SELECT (K301, de-energized = normal phase)"
- note added: "FINAL WET RETURN (never phase-flipped)"
- note added: "POWER + DECOUPLING"
- note added: "SIGNAL HEADERS"
- note removed: "Active stage"
- note removed: "Crossfade/feedback first-pass symbol capture - All required board refs are now present as real KiCad symbols - P307 is frozen as the current 10-pin grouped crossfade and feedback control landing - Crossfade summers, feedback polarity handling, and final wet-summing wiring still need the next capture pass"
- note removed: "Wet-loop headers"
