File: hardware/kicad/filter-clipper.kicad_sch (KiCad schematic)
At the start: 19 parts, among them P401 JXF-FILT, P402 JFILT-WET, P403 JFILT-CTL-A, P404 JFILT-PWR, P405 JFILT-CTL-B, U401 OPA1679IDR, U402 OPA1679IDR

Commit message: Board 4 filter-clipper: ERC 0, sim verified (HPF/drive 4.9x/clip modes/LPF), routed DRC 0/0, fab outputs; clip decode = 3x G5V-2 relay tree per frozen truth table
Parts:
- removed D405, D406, D407, D408: Clip LED, LED_SMD:LED_0805_2012Metric, symbol Device:D
- added C401, C421: 47n, Capacitor_SMD:C_1210_3225Metric, symbol Device:C
- added C403, C406, C407, C423, C426, C427: 10n, Capacitor_SMD:C_1210_3225Metric, symbol Device:C
- added C405, C425: 47p, Capacitor_SMD:C_0805_2012Metric, symbol Device:C
- added C591, C592, C593, C594: 100n, Capacitor_SMD:C_0805_2012Metric, symbol Device:C
- added C595, C596: 22u, Capacitor_SMD:C_1210_3225Metric, symbol Device:C
- added D405, D406, D407, D408: LED red, LED_SMD:LED_0805_2012Metric, symbol Device:LED
- added D421, D422: 1N4148W, Diode_SMD:D_SOD-123, symbol Device:D
- added K401, K402, K403: G5V-2 DC5, Relay_THT:Relay_DPDT_Omron_G5V-2, symbol Relay:G5V-2
- added R401, R406, R421, R426: 1k, Resistor_SMD:R_0805_2012Metric, symbol Device:R
- added R402, R407, R422, R427: 47k, Resistor_SMD:R_0805_2012Metric, symbol Device:R
- added R403, R423: 39k, Resistor_SMD:R_0805_2012Metric, symbol Device:R
- added R404, R424: 10k, Resistor_SMD:R_0805_2012Metric, symbol Device:R
- added R405, R425: 4.7k, Resistor_SMD:R_0805_2012Metric, symbol Device:R
- added R408, R428, R432: 100, Resistor_SMD:R_0805_2012Metric, symbol Device:R
- added unit 5 of U401
- added unit 3 of U401
- added unit 2 of U401
- added unit 4 of U401
- added unit 5 of U402
- added unit 4 of U402
- added unit 2 of U402
- added unit 3 of U402
- D401, D402, D403, D404: value 1N4148WS -> 1N4148W; footprint Diode_SMD:D_SOD-323 -> Diode_SMD:D_SOD-123
- D409, D410, D411, D412: value Ge clip or adapter -> 1N5819HW; footprint Diode_THT:D_DO-35_SOD27_P7.62mm_Horizontal -> Diode_SMD:D_SOD-123
- P401: value JXF-FILT -> JXF-FILT B3B-XH-A
- P402: value JFILT-WET -> JFILT-WET B3B-XH-A
- P403: value JFILT-CTL-A -> JFILT-CTL-A B12B-XH-A
- P404: value JFILT-PWR -> JFILT-PWR B3P-VH-B
- P405: value JFILT-CTL-B -> JFILT-CTL-B B12B-XH-A
Connections:
- net CTL_CLIP_MODE_A: now also P405.10 (Pin_10), D421.1 (K), K401.1
- net CTL_CLIP_MODE_B: now also P405.11 (Pin_11), D422.1 (K), K402.1, K403.1
- net DRV_HI: now also D401.1 (K), D402.2 (A), D403.1 (K), D404.2 (A), D409.1 (K), D410.2 (A), D411.1 (K), D412.2 (A), P403.1 (Pin_1), D405.1 (K), D406.2 (A), D407.1 (K), D408.2 (A)
- net DRV_WIPER: now also P403.2 (Pin_2), R432.1
- net FILTCLIP_OUT_L: now also P402.1 (Pin_1), R408.2
- net FILTCLIP_OUT_R: now also P402.3 (Pin_3), R428.2
- net HPF_F_L_HI: now also P403.4 (Pin_4), U401.3 (+), C401.2, C403.2
- net HPF_F_L_WIPER: now also P403.5 (Pin_5), R401.1
- net HPF_F_R_HI: now also P403.7 (Pin_7), C421.2, C423.2, U401.5 (+)
- net HPF_F_R_WIPER: now also P403.8 (Pin_8), R421.1
- net HPF_Q_L_WIPER: now also P403.10 (Pin_10), C403.1, R402.2
- net HPF_Q_R_WIPER: now also P403.11 (Pin_11), C423.1, R422.2
- net LPF_F_L_HI: now also P405.1 (Pin_1), R406.2
- net LPF_F_L_WIPER: now also P405.2 (Pin_2), U402.3 (+), C406.1, C407.2
- net LPF_F_R_HI: now also P405.4 (Pin_4), R426.2
- net LPF_F_R_WIPER: now also P405.5 (Pin_5), C426.1, C427.2, U402.5 (+)
- net LPF_Q_L_WIPER: now also P405.7 (Pin_7), C407.1, R407.2
- net LPF_Q_R_WIPER: now also P405.8 (Pin_8), C427.1, R427.2
- net XFADE_OUT_L: now also P401.1 (Pin_1), C401.1
- net XFADE_OUT_R: now also P401.3 (Pin_3), C421.1
- new net +15VA: C591.1, C593.1, C595.1, P404.1 (Pin_1), U401.4 (V+), U402.4 (V+)
- new net +5VAUX: P405.9 (Pin_9)
- new net -15VA: C592.1, C594.1, C596.1, P404.3 (Pin_3), U401.11 (V-), U402.11 (V-)
- new net AGND: C406.2, C426.2, C591.2, C592.2, C593.2, C594.2, C595.2, C596.2, D421.2 (A), D422.2 (A), K401.16, K402.16, K403.16, P401.2 (Pin_2), P402.2 (Pin_2), P403.12 (Pin_12), P403.3 (Pin_3), P403.6 (Pin_6), P403.9 (Pin_9), P404.2 (Pin_2), P405.12 (Pin_12), P405.3 (Pin_3), P405.6 (Pin_6), R401.2, R404.2, R421.2, R424.2, R432.2
- new net N_BUF_OUT_L: R408.1, U402.8, U402.9 (-)
- new net N_BUF_OUT_R: R428.1, U402.13 (-), U402.14
- new net N_CLIP_L: K401.4, R405.2, R406.1
- new net N_CLIP_R: K401.13, R425.2, R426.1
- new net N_DRV_M_L: C405.2, R403.2, R404.1, U401.9 (-)
- new net N_DRV_M_R: C425.2, R423.2, R424.1, U401.13 (-)
- new net N_DRV_OUT_L: C405.1, R403.1, R405.1, U401.8
- new net N_DRV_OUT_R: C425.1, R423.1, R425.1, U401.14
- new net N_GE_L: D409.2 (A), D410.1 (K), K402.9
- new net N_GE_R: D411.2 (A), D412.1 (K), K403.9
- new net N_HPF_OUT_L: R402.1, U401.1, U401.10 (+), U401.2 (-)
- new net N_HPF_OUT_R: R422.1, U401.12 (+), U401.6 (-), U401.7
- new net N_KA_L_NC: K401.6, K402.4
- new net N_KA_L_NO: K401.8, K402.13
- new net N_KA_R_NC: K401.11, K403.4
- new net N_KA_R_NO: K401.9, K403.13
- new net N_LED_L: D405.2 (A), D406.1 (K), K402.11
- new net N_LED_R: D407.2 (A), D408.1 (K), K403.11
- new net N_LPF_OUT_L: R407.1, U402.1, U402.10 (+), U402.2 (-)
- new net N_LPF_OUT_R: R427.1, U402.12 (+), U402.6 (-), U402.7
- new net N_SI_L: D401.2 (A), D402.1 (K), K402.8
- new net N_SI_R: D403.2 (A), D404.1 (K), K403.8
- no-connect marks 0 -> 2
Other:
- note added: "CLIP MODE DECODE (00 clean, 01 Si, 10 LED, 11 Schottky)"
- note added: "HEADERS"
- note added: "LEFT CHANNEL"
- note added: "POWER + DECOUPLING"
- note added: "RIGHT CHANNEL"
- note removed: "Active stages"
- note removed: "Audio and grouped control landings"
- note removed: "Clip networks"
- note removed: "Filter/clipper first-pass symbol capture - All required board refs are now present as real KiCad symbols - P403 and P405 follow the current 12-pin grouped-control split from the backplane definition - Germanium clip footprints are intentionally left provisional pending final device or adapter choice"
