File: hardware/kicad/filter-clipper.kicad_sch (KiCad schematic)
At the start: 19 parts, among them P401 JXF-FILT, P402 JFILT-WET, P403 JFILT-CTL-A, P404 JFILT-PWR, P405 JFILT-CTL-B, U401 OPA1679IDR, U402 OPA1679IDR

Commit message: Rev A: 3-pass schematic review + fixes, PCB sync + placement, parts freeze (2026-07-31)
Pass1+2 fixed cross-channel shorts (io rails/C1-C4/alias columns), ext-tank ghost wiring, U201 unit un-stack, U101-104 power units, PS500 pinout from datasheet, DRV renames. Decisions: TQ2-5V relays +D301, R241-3 deleted, PGND_IN+R502 link, K401-403 clip decoder, RCJ-041 tank jacks. GAS_Parts lib (TQ2/URA_YMD/RCJ-041), ~203 footprints, 6 boards synced+placed DRC-clean. Pass3 visual: paper sizes, stale notes. 3D GLBs + viewer. See hardware/kicad/schematic_review.md
Parts:
- added C401, C402, C421, C422, C471, C472, C491, C492: 22nF, Capacitor_SMD:C_0603_1608Metric, symbol Device:C
- added C591, C592, C593, C594: 100nF, Capacitor_SMD:C_0603_1608Metric, symbol Device:C
- added C595, C596: 10uF, Capacitor_SMD:CP_Elec_5x5.8, symbol Device:C
- added D421, D422: 1N4148, Diode_SMD:D_SOD-123, symbol Device:D
- added K401, K402, K403: TQ2-5V, GAS_Parts:Relay_DPDT_Panasonic_TQ2, symbol Relay:Relay_DPDT
- added R402, R422: 30k, Resistor_SMD:R_0603_1608Metric, symbol Device:R
- added R441, R442, R445, R446: 10k, Resistor_SMD:R_0603_1608Metric, symbol Device:R
- added R443, R444: 1k, Resistor_SMD:R_0603_1608Metric, symbol Device:R
- added R471, R491: 15k, Resistor_SMD:R_0603_1608Metric, symbol Device:R
- added R511, R512: 100R, Resistor_SMD:R_0603_1608Metric, symbol Device:R
- added unit 2 of U401
- added unit 3 of U401
- added unit 5 of U401
- added unit 4 of U401
- added unit 3 of U402
- added unit 2 of U402
- added unit 4 of U402
- added unit 5 of U402
- P405: Notes (none) -> RESOLVED 2026-07-31: clip-mode decode implemented as 3-rela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
Connections:
- net CTL_CLIP_MODE_A: now also P405.10 (Pin_10), D422.1 (K), K402.A1, K403.A1
- net CTL_CLIP_MODE_B: now also P405.11 (Pin_11), D421.1 (K), K401.A1
- net DRV_HI: now also P403.1 (Pin_1), R445.1, R446.1, U401.14, U401.8
- net DRV_WIPER: now also P403.2 (Pin_2), P403.3 (Pin_3), R441.1, R442.1, U401.13 (-), U401.9 (-)
- net FILTCLIP_OUT_L: now also P402.1 (Pin_1), R511.2
- net FILTCLIP_OUT_R: now also P402.3 (Pin_3), R512.2
- net HPF_F_L_HI: now also P403.4 (Pin_4), C401.2, C402.1
- net HPF_F_R_HI: now also P403.7 (Pin_7), C421.2, C422.1
- net HPF_Q_L_WIPER: now also P403.10 (Pin_10)
- net HPF_Q_R_WIPER: now also P403.11 (Pin_11)
- net LPF_F_L_HI: now also P405.1 (Pin_1)
- net LPF_F_R_HI: now also P405.4 (Pin_4)
- net LPF_Q_L_WIPER: now also P405.7 (Pin_7)
- net LPF_Q_R_WIPER: now also P405.8 (Pin_8)
- net XFADE_OUT_L: now also P401.1 (Pin_1), C401.1
- net XFADE_OUT_R: now also P401.3 (Pin_3), C421.1
- new net +15VA: C591.1, C593.1, C595.1, P404.1 (Pin_1), U401.4 (V+), U402.4 (V+)
- new net +5VAUX: P405.9 (Pin_9)
- new net -15VA: C592.1, C594.1, C596.1, P404.3 (Pin_3), U401.11 (V-), U402.11 (V-)
- new net AGND: C471.2, C491.2, C591.2, C592.2, C593.2, C594.2, C595.2, C596.2, D401.2 (A), D402.1 (K), D403.2 (A), D404.1 (K), D405.2 (A), D406.1 (K), D407.2 (A), D408.1 (K), D409.2 (A), D410.1 (K), D411.2 (A), D412.1 (K), D421.2 (A), D422.2 (A), K401.A2, K402.A2, K403.A2, P401.2 (Pin_2), P402.2 (Pin_2), P403.12 (Pin_12), P403.5 (Pin_5), P403.6 (Pin_6), P403.8 (Pin_8), P403.9 (Pin_9), P404.2 (Pin_2), P405.12 (Pin_12), R441.2, R442.2, U401.3 (+), U401.5 (+), U402.3 (+), U402.5 (+)
- new net BUF_OUT_L: R511.1, U402.8, U402.9 (-)
- new net BUF_OUT_R: R512.1, U402.13 (-), U402.14
- new net CLIP_NODE_L: K401.11, R445.2, R471.1
- new net CLIP_NODE_R: K401.21, R446.2, R491.1
- new net CLIP_W0_L: K401.12, K402.11
- new net CLIP_W0_R: K401.22, K402.21
- new net CLIP_W1_L: K401.14, K403.11
- new net CLIP_W1_R: K401.24, K403.21
- new net DRV_PRE_L: R443.2, U401.10 (+)
- new net DRV_PRE_R: R444.2, U401.12 (+)
- new net GE_CLIP_L: D409.1 (K), D410.2 (A), K403.14
- new net GE_CLIP_R: D411.1 (K), D412.2 (A), K403.24
- new net HPF_L_A: C402.2, R402.1, U401.2 (-)
- new net HPF_OUT_L: R402.2, R443.1, U401.1
- new net HPF_OUT_R: R422.2, R444.1, U401.7
- new net HPF_R_A: C422.2, R422.1, U401.6 (-)
- new net LED_CLIP_L: D405.1 (K), D406.2 (A), K402.14
- new net LED_CLIP_R: D407.1 (K), D408.2 (A), K402.24
- new net LPF_L_A: C472.1, P405.2 (Pin_2), P405.3 (Pin_3), U402.2 (-)
- new net LPF_N1_L: C471.1, R471.2
- new net LPF_N1_R: C491.1, R491.2
- new net LPF_OUT_L: C472.2, U402.1, U402.10 (+)
- new net LPF_OUT_R: C492.2, U402.12 (+), U402.7
- new net LPF_R_A: C492.1, P405.5 (Pin_5), P405.6 (Pin_6), U402.6 (-)
- new net SIL_CLIP_L: D401.1 (K), D402.2 (A), K403.12
- new net SIL_CLIP_R: D403.1 (K), D404.2 (A), K403.22
- no-connect marks 0 -> 2

Commit message: Rev A: asymmetric clipping - DNP D401/403/405/407/409/411 (sch+pcb+BOM), unify U401/U402 values, sheet note
Parts:
- D401, D403, D405, D407, D409, D411: now not fitted
- U401, U402: value OPA1679 -> OPA1679IDR
Other:
- note added: "Rev A build (2026-08-01): ASYMMETRIC clipping. D401 D403 D405 D407 D409 D411 are DNP (crossed out) - pads stay on the PCB. Remaining diode in each pair clips the POSITIVE half only -> even + odd harmonics. Populate the DNP pads to return any mode to symmetric clipping."
Changed lines of the file:
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@@
+		)
+	)
+	(text "Rev A build (2026-08-01): ASYMMETRIC clipping.\nD401 D403 D405 D407 D409 D411 are DNP (crossed out) - pads stay on the PCB.\nRemaining diode in each pair clips the POSITIVE half only -> even + odd harmonics.\nPopulate the DNP pads to return any mode to symmetric clipping."
+		(exclude_from_sim no)
+		(at 254.0 12.7 0)
+		(effects
+			(font
+				(size 1.8 1.8)
+			)
+			(justify left top)
 		)
 	)
@@
 		(on_board yes)
 		(in_pos_files yes)
-		(dnp no)
+		(dnp yes)
 		(fields_autoplaced yes)
 		(property "Reference" "D401"
@@
 		(on_board yes)
 		(in_pos_files yes)
-		(dnp no)
+		(dnp yes)
 		(fields_autoplaced yes)
 		(property "Reference" "D403"
@@
 		(on_board yes)
 		(in_pos_files yes)
-		(dnp no)
+		(dnp yes)
 		(fields_autoplaced yes)
 		(property "Reference" "D405"
@@
 		(on_board yes)
 		(in_pos_files yes)
-		(dnp no)
+		(dnp yes)
 		(fields_autoplaced yes)
 		(property "Reference" "D407"
@@
 		(on_board yes)
 		(in_pos_files yes)
-		(dnp no)
+		(dnp yes)
 		(fields_autoplaced yes)
 		(property "Reference" "D409"
@@
 		(on_board yes)
 		(in_pos_files yes)
-		(dnp no)
+		(dnp yes)
 		(fields_autoplaced yes)
 		(property "Reference" "D411"
@@
 			)
 		)
-		(property "Value" "OPA1679"
+		(property "Value" "OPA1679IDR"
 			(at 119.38 194.31 0)
 			(show_name no)
@@
 			)
 		)
-		(property "Value" "OPA1679"
+		(property "Value" "OPA1679IDR"
 			(at 119.38 234.95 0)
 			(show_name no)
@@
 			)
 		)
-		(property "Value" "OPA1679"
+		(property "Value" "OPA1679IDR"
 			(at 119.38 274.32 0)
 			(show_name no)
@@
 			)
 		)
-		(property "Value" "OPA1679"
+		(property "Value" "OPA1679IDR"
 			(at 119.38 314.96 0)
 			(show_name no)
@@
 			)
 		)
-		(property "Value" "OPA1679"
+		(property "Value" "OPA1679IDR"
 			(at 119.38 354.33 0)
 			(show_name no)
@@
 			)
 		)
-		(property "Value" "OPA1679"
+		(property "Value" "OPA1679IDR"
 			(at 119.38 394.97 0)
 			(show_name no)
@@
 			)
 		)
-		(property "Value" "OPA1679"
+		(property "Value" "OPA1679IDR"
 			(at 119.38 434.34 0)
 			(show_name no)
@@
 			)
 		)
-		(property "Value" "OPA1679"
+		(property "Value" "OPA1679IDR"
 			(at 119.38 474.98 0)
 			(show_name no)
