File: hardware/kicad/ext-tank-routing.kicad_sch (KiCad schematic)
At the start: 12 parts, among them K201 G6K-2F-Y-DC5, K202 G6K-2F-Y-DC5, K203 G6K-2F-Y-DC5, K204 G6K-2F-Y-DC5, P201 JIO-WETSEND, P202 JTR-PRI, P203 JTR-SEC, P204 JTR-XFADE, P205 JFB-INJ, P206 JER-CTRL, P207 JER-PWR, U201 OPA1679IDR

Commit message: Board 5 ext-tank-routing: ERC 0, sim verified (Series/Off relay modes, summers exact), routed DRC 0/0, fab outputs; relays standardized to G5V-2 DC5
Parts:
- removed K201, K202, K203, K204: G6K-2F-Y-DC5, Relay_SMD:Relay_DPDT_Omron_G6K-2F-Y, symbol Relay:Relay_DPDT
- added C291, C292, C295: 100n, Capacitor_SMD:C_0805_2012Metric, symbol Device:C
- added C293, C294: 22u, Capacitor_SMD:C_1210_3225Metric, symbol Device:C
- added D261, D262: 1N4148W, Diode_SMD:D_SOD-123, symbol Device:D
- added K201, K202, K203, K204: G5V-2 DC5, Relay_THT:Relay_DPDT_Omron_G5V-2, symbol Relay:G5V-2
- added R201, R205, R206, R221, R225, R226: 100, Resistor_SMD:R_0805_2012Metric, symbol Device:R
- added R202, R203, R204, R209, R222, R223, R224, R229, R241, R251: 20k, Resistor_SMD:R_0805_2012Metric, symbol Device:R
- added R211, R231: 100k, Resistor_SMD:R_0805_2012Metric, symbol Device:R
- added R212, R232: 0, Resistor_SMD:R_0805_2012Metric, symbol Device:R
- added unit 4 of U201
- added unit 2 of U201
- added unit 5 of U201
- added unit 3 of U201
- P201: value JIO-WETSEND -> P201
- P202: value JTR-PRI -> P202
- P203: value JTR-SEC -> P203
- P204: value JTR-XFADE -> P204
- P205: value JFB-INJ -> P205
- P206: value JER-CTRL -> P206
- P207: value JER-PWR -> P207
Connections:
- net +15VA: now also P207.1 (Pin_1), C291.1, C293.1, U201.4 (V+)
- net +5VAUX: now also P206.7 (Pin_7), P207.4 (Pin_4), C295.1
- net -15VA: now also P207.3 (Pin_3), C292.1, C294.1, U201.11 (V-)
- net AGND: now also P201.2 (Pin_2), P202.3 (Pin_3), P202.6 (Pin_6), P203.3 (Pin_3), P203.6 (Pin_6), P204.2 (Pin_2), P205.2 (Pin_2), P206.3 (Pin_3), P206.6 (Pin_6), P206.8 (Pin_8), P207.2 (Pin_2), U201.3 (+), C291.2, C292.2, C293.2, C294.2, C295.2, D261.2 (A), D262.2 (A), K201.16, K202.16, K203.16, K204.16, R211.2, R231.2, R241.2, R251.2, U201.5 (+)
- net CTL_EXT_MODE_A: now also P206.9 (Pin_9), D262.1 (K), K203.1, K204.1
- net CTL_EXT_MODE_B: now also P206.10 (Pin_10), D261.1 (K), K201.1, K202.1
- net EXTMIX_L_HI: now also P206.1 (Pin_1), K203.9
- net EXTMIX_L_WIPER: now also P206.2 (Pin_2), R203.1
- net EXTMIX_R_HI: now also P206.4 (Pin_4), K204.9
- net EXTMIX_R_WIPER: now also P206.5 (Pin_5), R223.1
- net FB_RET_L: now also P205.1 (Pin_1), R204.1
- net FB_RET_R: now also P205.3 (Pin_3), R224.1
- net PRI_RET_L: now also P202.2 (Pin_2), K201.6, R202.1
- net PRI_RET_R: now also P202.5 (Pin_5), K202.6, R222.1
- net PRI_SEND_L: now also P202.1 (Pin_1), R201.2
- net PRI_SEND_R: now also P202.4 (Pin_4), R221.2
- net SEC_DRV_L: now also K203.4, R211.1, U201.10 (+)
- net SEC_DRV_R: now also K204.4, R231.1, U201.12 (+)
- net SEC_RET_L: now also P203.2 (Pin_2), K203.13
- net SEC_RET_R: now also P203.5 (Pin_5), K204.13
- net SEC_SEL_L: now also K201.4, K203.8
- net SEC_SEL_R: now also K202.4, K204.8
- net SEC_SEND_L: now also P203.1 (Pin_1), R206.2
- net SEC_SEND_R: now also P203.4 (Pin_4), R226.2
- net TANK_MIX_L: now also P204.1 (Pin_1), R205.2
- net TANK_MIX_R: now also P204.3 (Pin_3), R225.2
- net WET_SEND_L: now also P201.1 (Pin_1), K201.8, R201.1
- net WET_SEND_R: now also P201.3 (Pin_3), K202.8, R221.1
- new net N_SECBUF_L: R206.1, R212.1, U201.8
- new net N_SECBUF_R: R226.1, R232.1, U201.14
- new net N_SECFB_L: R212.2, R241.1, U201.9 (-)
- new net N_SECFB_R: R232.2, R251.1, U201.13 (-)
- new net N_SUM_L_M: R202.2, R203.2, R204.2, R209.2, U201.2 (-)
- new net N_SUM_R_M: R222.2, R223.2, R224.2, R229.2, U201.6 (-)
- new net N_TMIX_L: R205.1, R209.1, U201.1
- new net N_TMIX_R: R225.1, R229.1, U201.7
- no-connect marks 0 -> 10
Other:
- note added: "FINAL SUMMERS"
- note added: "HEADERS"
- note added: "MODE RELAYS (A=engage, B=series/parallel)"
- note added: "POWER + DECOUPLING"
- note added: "PRIMARY SEND PASS-THROUGH"
- note added: "SECONDARY SEND BUFFERS"
- note removed: "Control and mode landing"
- note removed: "Ext-routing first-pass capture - All required board refs are present as real KiCad symbols - P206 remains frozen as the 10-pin JST XH control landing from the current connector schedule - Relay contact ownership, wet-send sheet ports, and connector net landings are now entered - Active summing, flyback support, and the full passive makeup network still need the next pass"
- note removed: "Inter-board headers"
- note removed: "Routing and buffer devices"

Commit message: ext-tank-routing: move feedback reinjection pre-tank (U202 send summers)
FB_RET_L/R now sum with WET_SEND_L/R at new OPA1656 send summers (U202)
upstream of PRI_SEND and the parallel-mode pickoff, so feedback re-passes
through the spring tanks. Removed FB_RET from the U201A/B TANK_MIX output
summers. Matches the JUCE sim, where feedbackReturnBuffer adds into
wetInputBaseBuffer before predelay+convolution (= the tanks).

- gen_ext.py: U202 stage, R207/R208/R227/R228 20k, C296/C297 100n,
  K201/K202 parallel contact now picks SEND_MIX; OPA1656 sim model added
- route_board.py: ext board routes AGND as a net (pour-only stranded
  U201 pad 5)
- ERC 0, tran sim verified (FB reaches PRI_SEND, absent from TANK_MIX),
  DRC 0 errors / 0 unconnected; fab packet regenerated
- docs: interfaces.md, ext-routing + crossfade schematic-ready defs,
  board doc, harness map, BOMs, order-readiness
Parts:
- removed D261, D262: 1N4148W, Diode_SMD:D_SOD-123, symbol Device:D
- removed R206, R226: 100, Resistor_SMD:R_0805_2012Metric, symbol Device:R
- removed R241: 20k, Resistor_SMD:R_0805_2012Metric, symbol Device:R
- removed unit 4 of U201
- added C296, C297: 100n, Capacitor_SMD:C_0805_2012Metric, symbol Device:C
- added R201: 100, Resistor_SMD:R_0805_2012Metric, symbol Device:R
- added R202, R203, R204, R207, R208, R222, R227, R228: 20k, Resistor_SMD:R_0805_2012Metric, symbol Device:R
- added R231: 100k, Resistor_SMD:R_0805_2012Metric, symbol Device:R
- added R232: 0, Resistor_SMD:R_0805_2012Metric, symbol Device:R
- added unit 3 of U202
- added unit 2 of U202
- D261: renamed from R231; value 100k -> 1N4148W; footprint Resistor_SMD:R_0805_2012Metric -> Diode_SMD:D_SOD-123; symbol Device:R -> Device:D
- D262: renamed from R232; value 0 -> 1N4148W; footprint Resistor_SMD:R_0805_2012Metric -> Diode_SMD:D_SOD-123; symbol Device:R -> Device:D
- R206: renamed from R203; value 20k -> 100
- R226: renamed from R222; value 20k -> 100
- R241: renamed from R202; now not fitted
- U201: renamed from R204; value 20k -> OPA1679IDR; footprint Resistor_SMD:R_0805_2012Metric -> Package_SO:SOIC-14_3.9x8.7mm_P1.27mm; symbol Device:R -> Amplifier_Operational:OPA1679
- U202: renamed from R201; value 100 -> OPA1656IDR; footprint Resistor_SMD:R_0805_2012Metric -> Package_SO:SOIC-8_3.9x4.9mm_P1.27mm; symbol Device:R -> Amplifier_Operational:OPA1656ID
Connections:
- net +15VA: now also C296.1, U202.8 (V+)
- net -15VA: now also C297.1, U202.4 (V-)
- net AGND: now also D262.2 (A), R241.2, U202.3 (+), C296.2, C297.2, R231.2, U202.5 (+)
- net CTL_EXT_MODE_A: now also D262.1 (K)
- net CTL_EXT_MODE_B: now also D261.1 (K)
- net EXTMIX_L_WIPER: now also R203.1; no longer R206.1
- net FB_RET_L: now also R204.1; no longer U201.1
- net N_SECBUF_L: now also R206.1
- net N_SECBUF_R: now also R226.1, U201.14, R232.1; no longer D262.1
- net N_SECFB_L: now also R241.1
- net N_SECFB_R: now also U201.13 (-), R232.2; no longer D262.2
- net N_SUM_L_M: now also R202.2, R203.2; no longer R206.2, R241.2, U201.2
- net N_SUM_R_M: now also R222.2; no longer R224.2, R226.2
- net PRI_RET_L: now also R202.1; no longer R241.1
- net PRI_RET_R: now also R222.1; no longer R226.1
- net PRI_SEND_L: now also R201.2; no longer U202.2
- net SEC_DRV_R: now also U201.12 (+), R231.1; no longer D261.1
- net SEC_SEND_L: now also R206.2
- net SEC_SEND_R: now also R226.2
- net WET_SEND_L: now also R207.1; no longer K201.8, U202.1
- net WET_SEND_R: now also R227.1; no longer K202.8, R221.1
- new net N_SND_L_M: R204.2, R207.2, R208.2, U202.2 (-)
- new net N_SND_R_M: R224.2, R227.2, R228.2, U202.6 (-)
- new net SEND_MIX_L: K201.8, R201.1, R208.1, U202.1
- new net SEND_MIX_R: K202.8, R221.1, R228.1, U202.7
Other:
- note added: "PRIMARY SEND (from send summers)"
- note added: "SEND SUMMERS (WET_SEND + FB_RET pre-tank reinjection)"
- note removed: "PRIMARY SEND PASS-THROUGH"
- moved on the sheet: R206, R226
