File: hardware/kicad/ext-tank-routing.kicad_sch (KiCad schematic)
At the start: 12 parts, among them K201 G6K-2F-Y-DC5, K202 G6K-2F-Y-DC5, K203 G6K-2F-Y-DC5, K204 G6K-2F-Y-DC5, P201 JIO-WETSEND, P202 JTR-PRI, P203 JTR-SEC, P204 JTR-XFADE, P205 JFB-INJ, P206 JER-CTRL, P207 JER-PWR, U201 OPA1679IDR

Commit message: Rev A: 3-pass schematic review + fixes, PCB sync + placement, parts freeze (2026-07-31)
Pass1+2 fixed cross-channel shorts (io rails/C1-C4/alias columns), ext-tank ghost wiring, U201 unit un-stack, U101-104 power units, PS500 pinout from datasheet, DRV renames. Decisions: TQ2-5V relays +D301, R241-3 deleted, PGND_IN+R502 link, K401-403 clip decoder, RCJ-041 tank jacks. GAS_Parts lib (TQ2/URA_YMD/RCJ-041), ~203 footprints, 6 boards synced+placed DRC-clean. Pass3 visual: paper sizes, stale notes. 3D GLBs + viewer. See hardware/kicad/schematic_review.md
Parts:
- added C291, C292, C295: 100nF, Capacitor_SMD:C_0603_1608Metric, symbol Device:C
- added C293, C294, C296: 10uF, Capacitor_SMD:CP_Elec_5x5.8, symbol Device:C
- added D261, D262, D263, D264: 1N4148W, Diode_SMD:D_SOD-123, symbol Device:D
- added R201, R205, R206, R221, R225, R226: 100R, Resistor_SMD:R_0603_1608Metric, symbol Device:R
- added R202, R203, R204, R209, R222, R223, R224, R229: 20k, Resistor_SMD:R_0603_1608Metric, symbol Device:R
- added R211, R231: 100k, Resistor_SMD:R_0603_1608Metric, symbol Device:R
- added unit 5 of U201
- added unit 4 of U201
- added unit 3 of U201
- added unit 2 of U201
- K201, K202: value G6K-2F-Y-DC5 -> TQ2-5V; footprint Relay_SMD:Relay_DPDT_Omron_G6K-2F-Y -> GAS_Parts:Relay_DPDT_Panasonic_TQ2; Alt_MPN (none) -> Substitutes MUST match TQ2 10-pin THT land pattern (HFD4/HF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; MPN (none) -> TQ2-5V; Notes (none) -> Coil driven directly by switched +5VAUX (CTL_EXT_MODE_B) pe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
- K203, K204: value G6K-2F-Y-DC5 -> TQ2-5V; footprint Relay_SMD:Relay_DPDT_Omron_G6K-2F-Y -> GAS_Parts:Relay_DPDT_Panasonic_TQ2; Alt_MPN (none) -> Substitutes MUST match TQ2 10-pin THT land pattern (HFD4/HF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; MPN (none) -> TQ2-5V; Notes (none) -> Coil driven directly by switched +5VAUX (CTL_EXT_MODE_A) pe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
- P206: Notes (none) -> RESOLVED 2026-07-31: (1) Relay coil direct drive confirmed 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
Connections:
- net +15VA: now also P207.1 (Pin_1), C291.1, C293.1, U201.4 (V+)
- net +5VAUX: now also P206.7 (Pin_7), P207.4 (Pin_4), C295.1, C296.1
- net -15VA: now also P207.3 (Pin_3), C292.1, C294.1, U201.11 (V-)
- net AGND: now also K201.A2, K202.A2, K203.12, K203.22, K203.A2, K204.12, K204.22, K204.A2, P201.2 (Pin_2), P202.3 (Pin_3), P202.6 (Pin_6), P203.3 (Pin_3), P203.6 (Pin_6), P204.2 (Pin_2), P205.2 (Pin_2), P206.3 (Pin_3), P206.6 (Pin_6), P206.8 (Pin_8), P207.2 (Pin_2), U201.3 (+), C291.2, C292.2, C293.2, C294.2, C295.2, C296.2, D261.2 (A), D262.2 (A), D263.2 (A), D264.2 (A), R211.2, R231.2, U201.5 (+)
- net CTL_EXT_MODE_A: now also K203.A1, K204.A1, P206.9 (Pin_9), D263.1 (K), D264.1 (K)
- net CTL_EXT_MODE_B: now also K201.A1, K202.A1, P206.10 (Pin_10), D261.1 (K), D262.1 (K)
- net EXTMIX_L_HI: now also K203.21, P206.1 (Pin_1)
- net EXTMIX_L_WIPER: now also P206.2 (Pin_2), R203.1
- net EXTMIX_R_HI: now also K204.21, P206.4 (Pin_4)
- net EXTMIX_R_WIPER: now also P206.5 (Pin_5), R223.1
- net FB_RET_L: now also P205.1 (Pin_1), R204.1
- net FB_RET_R: now also P205.3 (Pin_3), R224.1
- net PRI_RET_L: now also K201.12, P202.2 (Pin_2), R202.1
- net PRI_RET_R: now also K202.12, P202.5 (Pin_5), R222.1
- net PRI_SEND_L: now also P202.1 (Pin_1), R201.2
- net PRI_SEND_R: now also P202.4 (Pin_4), R221.2
- net SEC_DRV_L: now also K203.11, R211.1, U201.10 (+)
- net SEC_DRV_R: now also K204.11, R231.1, U201.12 (+)
- net SEC_RET_L: now also K203.24, P203.2 (Pin_2)
- net SEC_RET_R: now also K204.24, P203.5 (Pin_5)
- net SEC_SEL_L: now also K201.11, K203.14
- net SEC_SEL_R: now also K202.11, K204.14
- net SEC_SEND_L: now also P203.1 (Pin_1), R206.2
- net SEC_SEND_R: now also P203.4 (Pin_4), R226.2
- net TANK_MIX_L: now also P204.1 (Pin_1), R205.2
- net TANK_MIX_R: now also P204.3 (Pin_3), R225.2
- net WET_SEND_L: now also K201.14, P201.1 (Pin_1), R201.1
- net WET_SEND_R: now also K202.14, P201.3 (Pin_3), R221.1
- new net U201A_M: R202.2, R203.2, R204.2, R209.2, U201.2 (-)
- new net U201A_OUT: R205.1, R209.1, U201.1
- new net U201B_M: R222.2, R223.2, R224.2, R229.2, U201.6 (-)
- new net U201B_OUT: R225.1, R229.1, U201.7
- new net U201C_OUT: R206.1, U201.8, U201.9 (-)
- new net U201D_OUT: R226.1, U201.13 (-), U201.14
Other:
- note added: "Ext-routing first-pass capture - All required board refs are present as real KiCad symbols - P206 remains frozen as the 10-pin JST XH control landing from the current connector schedule - Relay contact ownership, wet-send sheet ports, and connector net landings are now entered - COMPLETE 2026-07-31: U201A-D un-stacked & wired, flybacks D261-D264, relay decode verified, ghost wiring removed (see s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"
- note removed: "Ext-routing first-pass capture - All required board refs are present as real KiCad symbols - P206 remains frozen as the 10-pin JST XH control landing from the current connector schedule - Relay contact ownership, wet-send sheet ports, and connector net landings are now entered - Active summing, flyback support, and the full passive makeup network still need the next pass"
