File: hardware/kicad/io-board.kicad_sch (KiCad schematic)
At the start: 50 parts, among them J1 NCJ6FI-S, J2 NCJ6FI-S, J3 NCJ6FI-S, J4 NCJ6FI-S, P1 JIO-PWR, P2 JIO-WETSEND, P3 JIO-WETRET, P4 JIO-DRY, P5 Wet/Dry control, P6 Mono switch, U1 OPA1644AIDR, U2 OPA1656IDR, U3 OPA1656IDR, U4 OPA1656IDR

Commit message: Rev A: 3-pass schematic review + fixes, PCB sync + placement, parts freeze (2026-07-31)
Pass1+2 fixed cross-channel shorts (io rails/C1-C4/alias columns), ext-tank ghost wiring, U201 unit un-stack, U101-104 power units, PS500 pinout from datasheet, DRV renames. Decisions: TQ2-5V relays +D301, R241-3 deleted, PGND_IN+R502 link, K401-403 clip decoder, RCJ-041 tank jacks. GAS_Parts lib (TQ2/URA_YMD/RCJ-041), ~203 footprints, 6 boards synced+placed DRC-clean. Pass3 visual: paper sizes, stale notes. 3D GLBs + viewer. See hardware/kicad/schematic_review.md
Parts:
- added R21, R22, R23, R24: 100R, Resistor_SMD:R_0603_1608Metric, symbol Device:R_Small
- P1: Notes (none) -> SESSION NOTES: 2026-07-30 fixed crossed DRY_L/DRY_R strays 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
Connections:
- net +15VA: now also C91.1, C93.1, C95.1, C97.1, P1.1 (Pin_1), U1.4 (V+), U2.8 (V+), U3.8 (V+), U4.8 (V+)
- net -15VA: now also C92.1, C94.1, C96.1, C98.1, P1.3 (Pin_3), U1.11 (V-), U2.4 (V-), U3.4 (V-), U4.4 (V-)
- net AGND: now also C1.2, C2.2, C3.2, C4.2, C91.2, C92.2, C93.2, C94.2, C95.2, C96.2, C97.2, C98.2, J1.1, J1.G, J1.S, J2.1, J2.G, J2.S, J3.1, J3.G, J3.S, J4.1, J4.G, J4.S, P1.2 (Pin_2), P2.2 (Pin_2), P3.2 (Pin_2), P4.2 (Pin_2), R14.2, R18.2, U2.3 (+), U2.5 (+), U3.5 (+), U4.5 (+)
- net DRY_L: now also P4.1 (Pin_1), R21.2
- net DRY_R: now also P4.3 (Pin_3), R23.2
- net IN_BAL_L_N: now also C2.1, J1.3, J1.R, R2.1
- net IN_BAL_L_P: now also C1.1, J1.2, J1.T, R1.1
- net IN_BAL_R_N: now also C4.1, J2.3, J2.R, R4.1
- net IN_BAL_R_P: now also C3.1, J2.2, J2.T, R3.1
- net L_BLEND: now also R35.1, R43.1, U2.1, U3.3 (+)
- net L_COLD_DRV: now also R44.1, R50.1, U3.7
- net L_HOT_DRV: now also R49.1, U3.1, U3.2 (-)
- net MONO_A: now also P6.1 (Pin_1), R12.1, U1.1, U1.10 (+)
- net MONO_B: now also P6.3 (Pin_3), R16.1, U1.7
- net MONO_C: now also P6.2 (Pin_2), U1.12 (+)
- net OUT_BAL_L_N: now also J3.3, J3.R, R50.2
- net OUT_BAL_L_P: now also J3.2, J3.T, R49.2
- net OUT_BAL_R_N: now also J4.3, J4.R, R60.2
- net OUT_BAL_R_P: now also J4.2, J4.T, R59.2
- net R_BLEND: now also R36.1, R53.1, U2.7, U4.3 (+)
- net R_COLD_DRV: now also R54.1, R60.1, U4.7
- net R_HOT_DRV: now also R59.1, U4.1, U4.2 (-)
- net U1A_P: now also R13.2, R14.1, U1.3 (+)
- net U1B_P: now also R17.2, R18.1, U1.5 (+)
- net WD_L_HI: now also P5.1 (Pin_1), U1.8, U1.9 (-), R21.1, R22.1
- net WD_L_LO: now also P3.1 (Pin_1), P5.3 (Pin_3)
- net WD_L_WIPER: now also P5.2 (Pin_2), R31.1
- net WD_R_HI: now also P5.4 (Pin_4), U1.13 (-), U1.14, R23.1, R24.1
- net WD_R_LO: now also P3.3 (Pin_3), P5.6 (Pin_6)
- net WD_R_WIPER: now also P5.5 (Pin_5), R32.1
- net WET_SEND_L: now also P2.1 (Pin_1), R22.2
- net WET_SEND_R: now also P2.3 (Pin_3), R24.2
- new net INBUF_L_N: R11.1, R2.2
- new net INBUF_L_P: R1.2, R13.1
- new net INBUF_R_N: R15.1, R4.2
- new net INBUF_R_P: R17.1, R3.2
- new net L_RX_M: R11.2, R12.2, U1.2 (-)
- new net R_RX_M: R15.2, R16.2, U1.6 (-)
- new net U2A_M: R31.2, R35.2, U2.2 (-)
- new net U2B_M: R32.2, R36.2, U2.6 (-)
- new net U3B_M: R43.2, R44.2, U3.6 (-)
- new net U4B_M: R53.2, R54.2, U4.6 (-)
