File: hardware/kicad/power-backplane.kicad_pcb (KiCad board)
At the start: 2 copper layers, 150 x 95 mm, 18 parts, among them P501 I/O board power, P502 Tank board power, P503 Crossfade board power, P504 Filter board power, P505 Spare utility power, P506 Ext-routing board power, P601 Control-backplane power

Commit message: Rev A: 3-pass schematic review + fixes, PCB sync + placement, parts freeze (2026-07-31)
Pass1+2 fixed cross-channel shorts (io rails/C1-C4/alias columns), ext-tank ghost wiring, U201 unit un-stack, U101-104 power units, PS500 pinout from datasheet, DRV renames. Decisions: TQ2-5V relays +D301, R241-3 deleted, PGND_IN+R502 link, K401-403 clip decoder, RCJ-041 tank jacks. GAS_Parts lib (TQ2/URA_YMD/RCJ-041), ~203 footprints, 6 boards synced+placed DRC-clean. Pass3 visual: paper sizes, stale notes. 3D GLBs + viewer. See hardware/kicad/schematic_review.md
Parts:
- added J500: PJ-005B, Connector_BarrelJack:BarrelJack_Horizontal, F.Cu at (14.0, 50.0)
- added PS500: URA2415YMD-10WR3, GAS_Parts:Converter_DCDC_Mornsun_URA_YMD_THT, F.Cu at (60.0, 50.0)
- added R502: 0R, Resistor_SMD:R_0603_1608Metric, F.Cu at (90.0, 45.0)
Connections:
- C500 pad 1: (no net) -> PGND_IN
- C500 pad 2: (no net) -> +30VIN
- D500 pad 1: (no net) -> VIN_FUSED
- D500 pad 2: (no net) -> +30VIN
- F500 pad 1: (no net) -> VIN_FUSED
- F500 pad 2: (no net) -> VIN_ENTRY
- FB500 pad 1: (no net) -> +15VA
- FB500 pad 2: (no net) -> +15V_RAW
- FB501 pad 1: (no net) -> -15VA
- FB501 pad 2: (no net) -> -15V_RAW
- P501 pad 1: (no net) -> -15VA
- P501 pad 2: (no net) -> AGND
- P501 pad 3: (no net) -> +15VA
- P502 pad 1: (no net) -> -15VA
- P502 pad 2: (no net) -> AGND
- P502 pad 3: (no net) -> +15VA
- P503 pad 1: (no net) -> -15VA
- P503 pad 2: (no net) -> AGND
- P503 pad 3: (no net) -> +15VA
- P504 pad 1: (no net) -> -15VA
- P504 pad 2: (no net) -> AGND
- P504 pad 3: (no net) -> +15VA
- P505 pad 1: (no net) -> -15VA
- P505 pad 2: (no net) -> AGND
- P505 pad 3: (no net) -> +15VA
- P506 pad 1: (no net) -> -15VA
- P506 pad 2: (no net) -> AGND
- P506 pad 3: (no net) -> +15VA
- P506 pad 4: (no net) -> +5VAUX
- P601 pad 1: (no net) -> +15VA
- P601 pad 2: (no net) -> AGND
- P601 pad 3: (no net) -> +5VAUX
- P601 pad 4: (no net) -> -15VA
- PS501 pad 1: (no net) -> +15VA
- PS501 pad 2: (no net) -> AGND
- PS501 pad 3: (no net) -> +5VAUX
- TVS500 pad 1: (no net) -> PGND_IN
- TVS500 pad 2: (no net) -> +30VIN
