File: hardware/kicad/power-backplane.kicad_sch (KiCad schematic)
At the start: 16 parts, among them J500 PJ-005B, P501 I/O board power, P502 Tank board power, P503 Crossfade board power, P504 Filter board power, P505 Spare utility power, P506 Ext-routing board power, P601 Control-backplane power

Commit message: Rev A: 3-pass schematic review + fixes, PCB sync + placement, parts freeze (2026-07-31)
Pass1+2 fixed cross-channel shorts (io rails/C1-C4/alias columns), ext-tank ghost wiring, U201 unit un-stack, U101-104 power units, PS500 pinout from datasheet, DRV renames. Decisions: TQ2-5V relays +D301, R241-3 deleted, PGND_IN+R502 link, K401-403 clip decoder, RCJ-041 tank jacks. GAS_Parts lib (TQ2/URA_YMD/RCJ-041), ~203 footprints, 6 boards synced+placed DRC-clean. Pass3 visual: paper sizes, stale notes. 3D GLBs + viewer. See hardware/kicad/schematic_review.md
Parts:
- added R502: 0R, Resistor_SMD:R_0603_1608Metric, symbol Device:R
- J500: footprint (none) -> Connector_BarrelJack:BarrelJack_Horizontal
- PS500: value URB2415YMD-10WR3 -> URA2415YMD-10WR3; footprint (none) -> GAS_Parts:Converter_DCDC_Mornsun_URA_YMD_THT; Alt_MPN (none) -> Approved alternates (same industry 1x1in package/pinout, 9-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; Notes (none) -> Pinout CONFIRMED 2026-07-31 from official Mornsun URA_YMD-1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
Connections:
- net +15VA: now also FB500.1, P501.3 (Pin_3), P502.3 (Pin_3), P503.3 (Pin_3), P504.3 (Pin_3), P505.3 (Pin_3), P506.3 (Pin_3), P601.1 (Pin_1), PS501.1 (IN)
- net +15V_RAW: now also FB500.2, PS500.3 (Pin_3)
- net +30VIN: now also C500.2, D500.2 (A), PS500.2 (Pin_2), TVS500.2 (A2)
- net +5VAUX: now also P506.4 (Pin_4), P601.3 (Pin_3), PS501.3 (OUT)
- net -15VA: now also FB501.1, P501.1 (Pin_1), P502.1 (Pin_1), P503.1 (Pin_1), P504.1 (Pin_1), P505.1 (Pin_1), P506.1 (Pin_1), P601.4 (Pin_4)
- net -15V_RAW: now also FB501.2, PS500.5 (Pin_5)
- net AGND: now also P501.2 (Pin_2), P502.2 (Pin_2), P503.2 (Pin_2), P504.2 (Pin_2), P505.2 (Pin_2), P506.2 (Pin_2), P601.2 (Pin_2), PS500.4 (Pin_4), PS501.2 (GND), R502.2
- net VIN_ENTRY: now also F500.2, J500.2
- net VIN_FUSED: now also D500.1 (K), F500.1
- new net PGND_IN: C500.1, J500.1, PS500.1 (Pin_1), R502.1, TVS500.1 (A1)
Other:
- note added: "Power-backplane first-pass electrical capture - DC entry, split-rail generation, and board harness outputs are now net-assigned - Global project rails remain anchored for ERC visibility - 2026-07-31: PS500 pinout datasheet-confirmed; PGND_IN input-ground island + R502 0R link added; chassis-bond network intentionally minimal (revisit at enclosure build)"
- note removed: "Power-backplane first-pass electrical capture - DC entry, split-rail generation, and board harness outputs are now net-assigned - Global project rails remain anchored for ERC visibility - Post-conversion ripple-decoupling parts and the controlled chassis-bond network still need the next capture pass"
