File: hardware/kicad/sim/ext-tank-routing-sim/ext-tank-routing-sim.kicad_sch (KiCad schematic)
At the start: 61 parts, among them K201 G5V-2 DC5, K202 G5V-2 DC5, K203 G5V-2 DC5, K204 G5V-2 DC5, P201 P201, P202 P202, P203 P203, P204 P204, P205 P205, P206 P206, P207 P207, U201 OPA1679IDR

Commit message: ext-tank-routing: move feedback reinjection pre-tank (U202 send summers)
FB_RET_L/R now sum with WET_SEND_L/R at new OPA1656 send summers (U202)
upstream of PRI_SEND and the parallel-mode pickoff, so feedback re-passes
through the spring tanks. Removed FB_RET from the U201A/B TANK_MIX output
summers. Matches the JUCE sim, where feedbackReturnBuffer adds into
wetInputBaseBuffer before predelay+convolution (= the tanks).

- gen_ext.py: U202 stage, R207/R208/R227/R228 20k, C296/C297 100n,
  K201/K202 parallel contact now picks SEND_MIX; OPA1656 sim model added
- route_board.py: ext board routes AGND as a net (pour-only stranded
  U201 pad 5)
- ERC 0, tran sim verified (FB reaches PRI_SEND, absent from TANK_MIX),
  DRC 0 errors / 0 unconnected; fab packet regenerated
- docs: interfaces.md, ext-routing + crossfade schematic-ready defs,
  board doc, harness map, BOMs, order-readiness
Parts:
- removed P203: P203, Connector_JST:JST_XH_B6B-XH-A_1x06_P2.50mm_Vertical, symbol Connector_Generic:Conn_01x06
- removed P205: P205, Connector_JST:JST_XH_B3B-XH-A_1x03_P2.50mm_Vertical, symbol Connector_Generic:Conn_01x03
- removed V1, V2: 15V, symbol Simulation_SPICE:VDC
- added C296, C297: 100n, Capacitor_SMD:C_0805_2012Metric, symbol Device:C
- added K201: G5V-2 DC5, Relay_THT:Relay_DPDT_Omron_G5V-2, symbol Relay:G5V-2
- added P207: P207, Connector_JST:JST_VH_B4P-VH_1x04_P3.96mm_Vertical, symbol Connector_Generic:Conn_01x04
- added R207, R208, R227, R228: 20k, Resistor_SMD:R_0805_2012Metric, symbol Device:R
- added RL4, RL5: 10k, Resistor_SMD:R_0805_2012Metric, symbol Device:R
- added U202: OPA1656IDR, Package_SO:SOIC-8_3.9x4.9mm_P1.27mm, symbol Amplifier_Operational:OPA1656ID
- P203: renamed from P207; value P207 -> P203; footprint Connector_JST:JST_VH_B4P-VH_1x04_P3.96mm_Vertical -> Connector_JST:JST_XH_B6B-XH-A_1x06_P2.50mm_Vertical; symbol Connector_Generic:Conn_01x04 -> Connector_Generic:Conn_01x06
- P205: renamed from K201; value G5V-2 DC5 -> P205; footprint Relay_THT:Relay_DPDT_Omron_G5V-2 -> Connector_JST:JST_XH_B3B-XH-A_1x03_P2.50mm_Vertical; symbol Relay:G5V-2 -> Connector_Generic:Conn_01x03
- V1: renamed from RL4; value 10k -> 15V; footprint Resistor_SMD:R_0805_2012Metric -> (none); symbol Device:R -> Simulation_SPICE:VDC
- V2: renamed from RL5; value 10k -> 15V; footprint Resistor_SMD:R_0805_2012Metric -> (none); symbol Device:R -> Simulation_SPICE:VDC
Connections:
- net +15VA: now also V1.1, C296.1, P207.1 (Pin_1), U202.8 (V+); no longer P203.1 (Pin_1)
- net +5VAUX: now also P207.4 (Pin_4); no longer P203.4 (Pin_4)
- net -15VA: now also V2.2, C297.1, P207.3 (Pin_3), U202.4 (V-); no longer P203.3 (Pin_3)
- net AGND: now also P203.3 (Pin_3), P203.6 (Pin_6), P205.2 (Pin_2), C296.2, C297.2, K201.16, P207.2 (Pin_2), RL4.2, RL5.2, U202.3 (+), U202.5 (+); no longer P203.2 (Pin_2), P205.16, V1.2, V2.2
- net CTL_EXT_MODE_B: now also K201.1; no longer P205.1
- net FB_RET_L: now also P205.1 (Pin_1)
- net FB_RET_R: now also P205.3 (Pin_3)
- net GND: now also V1.2, V2.1
- net N_SUM_L_M: no longer R204.2
- net N_SUM_R_M: no longer R224.2
- net PRI_RET_L: now also K201.6; no longer P205.6
- net PRI_SEND_L: now also RL5.1; no longer V2.1
- net SEC_RET_L: now also P203.2 (Pin_2)
- net SEC_RET_R: now also P203.5 (Pin_5)
- net SEC_SEL_L: now also K201.4; no longer P205.4
- net SEC_SEND_L: now also P203.1 (Pin_1)
- net SEC_SEND_R: now also P203.4 (Pin_4), RL4.1; no longer V1.1
- net WET_SEND_L: now also R207.1; no longer P205.8, R201.1
- net WET_SEND_R: now also R227.1; no longer K202.8, R221.1
- new net N_SND_L_M: R204.2, R207.2, R208.2, U202.2 (-)
- new net N_SND_R_M: R224.2, R227.2, R228.2, U202.6 (-)
- new net SEND_MIX_L: K201.8, R201.1, R208.1, U202.1
- new net SEND_MIX_R: K202.8, R221.1, R228.1, U202.7
Other:
- note added: "PRIMARY SEND (from send summers)"
- note added: "SEND SUMMERS (WET_SEND + FB_RET pre-tank reinjection)"
- note removed: "PRIMARY SEND PASS-THROUGH"
