File: hardware/kicad/revc/circuit-board/circuit-board.kicad_sch (KiCad schematic)
At the start: 242 parts, among them K1 G6K-2F-Y DC5, K2 G6K-2F-Y DC5, K3 G6K-2F-Y DC5, K4 G6K-2F-Y DC5, K5 G6K-2F-Y DC5, P1 TANK-RET (from tank board), P2 WET-OUT (to io-board), P3 FB-RET (to tank board), P4 PWR (from power board), P5 CTL-A: HPF quad 50k lin (PTD9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, P6 CTL-B: LPF quad 50k lin (PTD9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, P7 CTL-C: Ext Mix dual 10k lin, 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, P8 CTL-D: switch lines (from con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, P9 CTL-E: Gain dual 10k lin (con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, Q1201 MMBF5457, Q1221 MMBF5457, Q1341 MMBT3906, U101 L78L09, U102 TL072HIDR, U1201 OPA1679IDR, U1301 OPA1679IDR, U1302 OPA1679IDR, U1303 V2181, U1304 V2181, U1305 OPA1679IDR, U201 OPA1679IDR, U202 OPA1679IDR, U301 OPA1679IDR, U302 OPA1679IDR, U402 TL072HIDR

Commit message: Rev C: Comp/Limit into the feedback return leg, per-mode tank blend knob
Plugin (signal-path diagram v4/v5, 2026-09-30):

- Comp / Off / Limit moves out of the wet path and into the feedback RETURN
  leg, between the Feedback Fb% block and the Fb In summer, so its job is
  holding the loop down rather than shaping what you hear. New
  FeedbackDynamicsBlock carries the circuit plus its oversampling; the wet
  path's DirtDynamicsBlock now always runs Dynamics::off.
- Both thresholds drop 6 dB, kThresholdDbfs -18 -> -24 dBFS, so there is
  something to grab with before the loop is already loud.
- Comp is the MMBF5457 FET model (refs 12xx), not the VTL5C3 vactrol; the
  limiter is a Coolaudio V2181. Stale tooltips corrected.
- Tank blend knob is now per routing: N/A and greyed out in Off, "+ %Long
  Tank" 0-100% linear in Series, "Short / Long Tank Mix" reading
  "x% Short / 100-x% Long" in Parallel. Host automation text matches.
- Per-lane wet predelay ranges (20-30 / 22-35 / 30-42 / 25-40 ms).
- Chain readout: "Fb Out + Comp" / "+ Lim", "In: Tube", and
  "Out: Tube & Tape" so the output tube is visible. The Out knob label only
  looked at Tape before, so it read "Out: Solid State" with the tube in.

Hardware:

- circuit-board re-netted so HPF precedes Gain, matching the schematic
  annotation; ERC 0, Freerouting clean, DRC 0 unconnected / 0 parity.
- U1303/U1304 are Coolaudio V2181; RV1301/RV1321 symmetry trims fitted.
- Fab exports and docs refreshed; rev-c-hardware-definition.md is the live
  spec, the 09-16 PCB release doc stays as the historical record.
- Signal-path draw.io lineage added (v2 through v5).

Repo hygiene:

- .gitignore now covers the cmake-out trees (~1 GB), agent scratch scripts
  and editor .bak files.
- The origin remote no longer carries an embedded personal access token.

Co-Authored-By: Claude Opus 5 <noreply@anthropic.com>
Claude-Session: https://claude.ai/code/session_01CUj6HcY7Ru31X8UWN7atuH
Connections:
- net AGND: now also U201.10 (+), U301.10 (+); no longer U201.5 (+), U301.5 (+)
- net GAIN_L_W: now also U201.9 (-); no longer U201.6 (-)
- net GAIN_OUT_L: now also K1.2, R215.1, U201.8; no longer C202.1, C212.1, U201.7
- net GAIN_OUT_R: now also K1.7, R315.1, U301.8; no longer C302.1, C312.1, U301.7
- net GAIN_R_W: now also U301.9 (-); no longer U301.6 (-)
- net HPF_FB_L: now also U201.6 (-); no longer U201.9 (-)
- net HPF_FB_R: now also U301.6 (-); no longer U301.9 (-)
- net HPF_OUT_L: now also R201.1, U201.7; no longer K1.2, R215.1, U201.8
- net HPF_OUT_R: now also R301.1, U301.7; no longer K1.7, R315.1, U301.8
- net HPF_P_L: now also U201.5 (+); no longer U201.10 (+)
- net HPF_P_R: now also U301.5 (+); no longer U301.10 (+)
- net TANK_MIX_L: now also C202.1, C212.1; no longer R201.1
- net TANK_MIX_R: now also C302.1, C312.1; no longer R301.1
Other:
- note added: "Main path L: Ext Mix sum, HPF, Gain, LPF"
- note added: "Main path R: Ext Mix sum, HPF, Gain, LPF"
- note removed: "Main path L: Ext Mix sum, Gain, HPF, LPF"
- note removed: "Main path R: Ext Mix sum, Gain, HPF, LPF"
- moved on the sheet: C201, C202, C203, C212, C213, C301, C302, C303, C312, C313, R201, R202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
